File: flip-pixel.sch (KiCad schematic (older format))
At the start: 19 parts, among them J1 Barrel-Jack, Q1 DMN62D0U-7, U1 LM2665M6, U2 ESP32_DevBoard, U3 INA250A3

Commit message: Began work on 0.2
Parts:
- added U? (x3): NPIC6C596ADJ, symbol Custom-Symbols:NPIC6C596ADJ
- C1, C2, C3, C4, C5: symbol Device:C -> flip-pixel-rescue:C-Device
- D1: symbol Custom-Symbols:Diode -> flip-pixel-rescue:Diode-Custom-Symbols
- D52, D53: symbol Custom-Symbols:LED_Green -> flip-pixel-rescue:LED_Green-Custom-Symbols
- J1: symbol Custom-Symbols:Barrel-Jack -> flip-pixel-rescue:Barrel-Jack-Custom-Symbols
- JP1: symbol Jumper:SolderJumper_2_Open -> flip-pixel-rescue:SolderJumper_2_Open-Jumper
- LOGO1: symbol Graphic:Logo_Open_Hardware_Small -> flip-pixel-rescue:Logo_Open_Hardware_Small-Graphic
- Q1: symbol Custom-Symbols:DMN62D0U-7 -> flip-pixel-rescue:DMN62D0U-7-Custom-Symbols
- R1, R2, R23, R24: symbol Device:R -> flip-pixel-rescue:R-Device
- U1: symbol Custom-Symbols:LM2665M6 -> flip-pixel-rescue:LM2665M6-Custom-Symbols
- U2: symbol Custom-Symbols:ESP32_DevBoard -> flip-pixel-rescue:ESP32_DevBoard-Custom-Symbols
- U3: symbol Custom-Symbols:INA250A3 -> flip-pixel-rescue:INA250A3-Custom-Symbols
Connections:
- wire segments 200 -> 115
