File: flip-pixel.sch (KiCad schematic (older format))
At the start: 18 parts, among them J1 Barrel-Jack, Q1 DMN62D0U-7, U1 LM2665M6, U2 ESP32_DevBoard, U3 INA250A3

Commit message: Logos and SilkScreen
Parts:
- added LOGO1: Logo_Open_Hardware_Small, Symbol:OSHW-Logo2_9.8x8mm_SilkScreen, symbol Graphic:Logo_Open_Hardware_Small
Changed lines of the file:
@@
 Wire Bus Line
 	10300 3100 10300 6150
+$Comp
+L Graphic:Logo_Open_Hardware_Small LOGO1
+U 1 1 5F2FC01C
+P 5350 7200
+F 0 "LOGO1" H 5597 7225 50  0000 L CNN
+F 1 "Logo_Open_Hardware_Small" H 5350 6975 50  0001 C CNN
+F 2 "Symbol:OSHW-Logo2_9.8x8mm_SilkScreen" H 5350 7200 50  0001 C CNN
+F 3 "~" H 5350 7200 50  0001 C CNN
+	1    5350 7200
+	1    0    0    -1
+$EndComp
 $EndSCHEMATC

Commit message: changed files
Parts:
- removed C1, C2, C3, C5: C, Capacitor_SMD:C_0805_2012Metric, symbol Device:C
- removed C4: 0.1uF, Capacitor_SMD:C_0805_2012Metric, symbol Device:C
- removed D1: Diode, Diode_SMD:D_SOD-123F, symbol Custom-Symbols:Diode
- removed D52, D53: LED_Green, LED_SMD:LED_0805_2012Metric_Pad1.15x1.40mm_HandSolder, symbol Custom-Symbols:LED_Green
- removed JP1: BypassJumper, Jumper:SolderJumper-2_P1.3mm_Open_RoundedPad1.0x1.5mm, symbol Jumper:SolderJumper_2_Open
- removed Q1: DMN62D0U-7, Package_TO_SOT_SMD:SOT-23, symbol Custom-Symbols:DMN62D0U-7
- removed R1, R2, R23, R24: R, Resistor_SMD:R_0805_2012Metric, symbol Device:R
- removed U1: LM2665M6, Package_TO_SOT_SMD:SOT-23-6, symbol Custom-Symbols:LM2665M6
- removed U2: ESP32_DevBoard, Custom-Footprints:DIP-38_900_ELL, symbol Custom-Symbols:ESP32_DevBoard
- removed U3: INA250A3, Package_SO:TSSOP-16_4.4x5mm_P0.65mm, symbol Custom-Symbols:INA250A3
- added J2: USB_B_Micro, Connector_USB:USB_Micro-B_Amphenol_10103594-0001LF_Horizontal, symbol Connector:USB_B_Micro
Connections:
- net Power_Input is gone; now on net +5V: J1.1
- net GND: now also J2.5 (GND), J2.6 (Shield)
- new net Controller/usb_D+: J2.3 (D+)
- new net Controller/usb_D-: J2.2 (D-)
- no-connect marks 9 -> 2
Other:
- note removed: "Bypass Cap\nNear U3"
- note removed: "Charge Pump Voltage Doubler\n"
- note removed: "Filter Cap\nNear U3"
- note removed: "Pull Down\nResistor"
- note removed: "enable signal enables the high current\noperation of the pixel matrix by\ndriving the charge pump's\nshutdown pin low"
- moved on the sheet: J1, LOGO1

Commit message: All traces routed
Parts:
- removed J2: USB_B_Micro, Connector_USB:USB_Micro-B_Amphenol_10103594-0001LF_Horizontal, symbol Connector:USB_B_Micro
- added J2: MicroUSB, Custom-Footprints:USB_Micro-B_Amphenol_10104110_Horizontal, symbol Custom-Symbols:MicroUSB
Connections:
- net Controller/usb_D+: now also J2.3 (D+)
- net Controller/usb_D-: now also J2.2 (D-)
- net GND: now also J2.5 (GND), J2.6 (Shield)
Changed lines of the file:
@@
-	1    0    0    -1
-$EndComp
-$Comp
-L Connector:USB_B_Micro J2
-U 1 1 5F8E38C9
-P 1100 4000
-F 0 "J2" H 800 4350 50  0000 C CNN
-F 1 "USB_B_Micro" H 1100 4350 50  0000 C CNN
-F 2 "Connector_USB:USB_Micro-B_Amphenol_10103594-0001LF_Horizontal" H 1250 3950 50  0001 C CNN
-F 3 "~" H 1250 3950 50  0001 C CNN
-	1    1100 4000
 	1    0    0    -1
 $EndComp
@@
 Wire Bus Line
 	2950 4300 2950 6500
+Text Label 5500 3450 2    50   ~ 0
+MatrixControl1
 Text Label 5500 3350 2    50   ~ 0
-MatrixControl1
-Text Label 5500 3450 2    50   ~ 0
 MatrixControl2
 Text Label 5500 4000 2    50   ~ 0
@@
 Wire Wire Line
 	4750 6350 5550 6350
-Wire Bus Line
-	2950 6500 10250 6500
-Wire Bus Line
-	10350 3400 10350 6400
-Wire Bus Line
-	4800 3450 4800 6400
 Text Label 9650 3400 0    50   ~ 0
 MatrixControl12
@@
 Text Label 9650 6000 0    50   ~ 0
 MatrixControl20
+Wire Bus Line
+	2950 6500 10250 6500
+Wire Bus Line
+	10350 3400 10350 6400
+Wire Bus Line
+	4800 3450 4800 6400
+$Comp
+L Custom-Symbols:MicroUSB J2
+U 1 1 5FA3CEF5
+P 1100 4050
+F 0 "J2" H 950 4500 50  0000 C CNN
+F 1 "MicroUSB" H 1200 4500 50  0000 C CNN
+F 2 "Custom-Footprints:USB_Micro-B_Amphenol_10104110_Horizontal" H 1350 4450 50  0001 C CNN
+F 3 "https://www.amphenol-icc.com/media/wysiwyg/files/drawing/10118192.pdf" H 1350 4450 50  0001 C CNN
+F 4 "Digikey" H 900 4700 50  0001 C CNN "Vendor"
+F 5 "609-5379-1-ND" H 1150 4600 50  0001 C CNN "Vendor Part"
+F 6 "Amphenol ICC (FCI)" H 1150 4600 50  0001 C CNN "Manufacturer"
+F 7 "10118192-0002LF" H 1150 4600 50  0001 C CNN "Manufacture Part"
+	1    1100 4050
+	1    0    0    -1
+$EndComp
 $EndSCHEMATC

Commit message: Ready for Manufacture
Parts:
- added H1, H2, H3, H4: MountingHole, MountingHole:MountingHole_3mm, symbol Mechanical:MountingHole
Changed lines of the file:
@@
 Sheet 1 14
 Title "Flip Pixel Board"
-Date "2020-06-26"
-Rev ""
+Date "2020-09-14"
+Rev "0.2"
 Comp ""
 Comment1 ""
@@
 F1 "microcontroller.sch" 50
 F2 "matrix_enable" O R 2800 4050 50
-F3 "current" I R 2800 4150 50
+F3 "matrix_current" I R 2800 4150 50
 F4 "usb_D+" B L 1700 4000 50
 F5 "usb_D-" B L 1700 4100 50
@@
 MatrixControl11
 Wire Wire Line
-	5300 6350 5550 6350
-Wire Wire Line
 	4750 6350 5550 6350
 Text Label 9650 3400 0    50   ~ 0
@@
 Text Label 9650 6000 0    50   ~ 0
 MatrixControl20
-Wire Bus Line
-	2950 6500 10250 6500
-Wire Bus Line
-	10350 3400 10350 6400
-Wire Bus Line
-	4800 3450 4800 6400
 $Comp
 L Custom-Symbols:MicroUSB J2
@@
 	1    0    0    -1
 $EndComp
+Wire Bus Line
+	2950 6500 10250 6500
+Wire Bus Line
+	10350 3400 10350 6400
+Wire Bus Line
+	4800 3450 4800 6400
+$Comp
+L Mechanical:MountingHole H3
+U 1 1 5F637D31
+P 9050 850
+F 0 "H3" H 9150 896 50  0000 L CNN
+F 1 "MountingHole" H 9150 805 50  0000 L CNN
+F 2 "MountingHole:MountingHole_3mm" H 9050 850 50  0001 C CNN
+F 3 "~" H 9050 850 50  0001 C CNN
+	1    9050 850
+	1    0    0    -1
+$EndComp
+$Comp
+L Mechanical:MountingHole H1
+U 1 1 5F638D2C
+P 8200 850
+F 0 "H1" H 8300 896 50  0000 L CNN
+F 1 "MountingHole" H 8300 805 50  0000 L CNN
+F 2 "MountingHole:MountingHole_3mm" H 8200 850 50  0001 C CNN
+F 3 "~" H 8200 850 50  0001 C CNN
+	1    8200 850
+	1    0    0    -1
+$EndComp
+$Comp
+L Mechanical:MountingHole H2
+U 1 1 5F638FF0
+P 8200 1150
+F 0 "H2" H 8300 1196 50  0000 L CNN
+F 1 "MountingHole" H 8300 1105 50  0000 L CNN
+F 2 "MountingHole:MountingHole_3mm" H 8200 1150 50  0001 C CNN
+F 3 "~" H 8200 1150 50  0001 C CNN
+	1    8200 1150
+	1    0    0    -1
+$EndComp
+$Comp
+L Mechanical:MountingHole H4
+U 1 1 5F639222
+P 9050 1150
+F 0 "H4" H 9150 1196 50  0000 L CNN
+F 1 "MountingHole" H 9150 1105 50  0000 L CNN
+F 2 "MountingHole:MountingHole_3mm" H 9050 1150 50  0001 C CNN
+F 3 "~" H 9050 1150 50  0001 C CNN
+	1    9050 1150
+	1    0    0    -1
+$EndComp
