File: HalfBridge.sch (KiCad schematic (older format))
At the start: 9 parts, among them Q20 DMN62D0U-7, Q21 DMN62D0U-7, Q4 STS8DN6LF6AG

Commit message: Began work on 0.2
Parts:
- R3, R4, R41, R42: symbol Device:R -> flip-pixel-rescue:R-Device
Changed lines of the file:
@@
 $EndDescr
 $Comp
-L power:GND #PWR?
+L flip-pixel-rescue:GND-power #PWR?
 U 1 1 5EE9876D
 P 3800 3450
@@
 $EndComp
 $Comp
-L Device:R R?
+L flip-pixel-rescue:R-Device R?
 U 1 1 5EE98773
 P 3800 2800
@@
 $EndComp
 $Comp
-L power:GND #PWR?
+L flip-pixel-rescue:GND-power #PWR?
 U 1 1 5EE98786
 P 3800 4850
@@
 $EndComp
 $Comp
-L Device:R R?
+L flip-pixel-rescue:R-Device R?
 U 1 1 5EE9878C
 P 3800 4200
@@
 	4600 4200 4600 4100
 $Comp
-L power:GND #PWR?
+L flip-pixel-rescue:GND-power #PWR?
 U 1 1 5EE987B3
 P 4600 4600
@@
 	3800 4400 3800 4450
 $Comp
-L power:+5V #PWR060
+L flip-pixel-rescue:+5V-power #PWR060
 U 1 1 5F3ABF0C
 P 4600 2600
@@
 $EndComp
 $Comp
-L Device:R R?
+L flip-pixel-rescue:R-Device R?
 U 1 1 5F3B0E72
 P 7400 3600
@@
 $EndComp
 $Comp
-L power:GND #PWR?
+L flip-pixel-rescue:GND-power #PWR?
 U 1 1 5F3B0E78
 P 7400 3750
@@
 $EndComp
 $Comp
-L Device:R R?
+L flip-pixel-rescue:R-Device R?
 U 1 1 5F3B0E8B
 P 7850 3600
@@
 $EndComp
 $Comp
-L power:GND #PWR?
+L flip-pixel-rescue:GND-power #PWR?
 U 1 1 5F3B0E91
 P 7850 3750
