File: HalfBridge.sch (KiCad schematic (older format))
At the start: 3 parts, among them Q4 STS8DN6LF6AG

Commit message: more layout work
Connections:
- net High_ctl_OD renamed High_ctl
- net Low_ctl_OD renamed Low_ctl
- net PowerRail renamed MatrixPower
Changed lines of the file:
@@
 $Descr A 11000 8500
 encoding utf-8
-Sheet 3 14
+Sheet 9 14
 Title "Flip Pixel Board"
 Date "2020-06-20"
@@
 AR Path="/5EEA5FAB/5EE98773" Ref="R19"  Part="1"
 AR Path="/5EEA5FB2/5EE98773" Ref="R21"  Part="1"
-F 0 "R3" H 5500 2600 50  0000 R CNN
+F 0 "R15" H 5500 2600 50  0000 R CNN
 F 1 "R" H 5450 2500 50  0000 R CNN
 F 2 "Resistor_SMD:R_0805_2012Metric" V 5230 2550 50  0001 C CNN
@@
 AR Path="/5EEA5FAB/5EE9878C" Ref="R20"  Part="1"
 AR Path="/5EEA5FB2/5EE9878C" Ref="R22"  Part="1"
-F 0 "R4" H 5500 3550 50  0000 R CNN
+F 0 "R16" H 5500 3550 50  0000 R CNN
 F 1 "R" H 5450 3450 50  0000 R CNN
 F 2 "Resistor_SMD:R_0805_2012Metric" V 5230 3500 50  0001 C CNN
@@
 AR Path="/5EEA5FAB/5EE9879E" Ref="Q28"  Part="1"
 AR Path="/5EEA5FB2/5EE9879E" Ref="Q31"  Part="1"
-F 0 "Q4" H 6244 2796 50  0000 L CNN
+F 0 "Q22" H 6244 2796 50  0000 L CNN
 F 1 "STS8DN6LF6AG" H 6244 2705 50  0000 L CNN
 F 2 "Custom-Footprints:SO-8_3.9x4.9mm_P1.27mm" H 5750 3250 50  0001 C CNN
@@
 AR Path="/5EEA5FAB/5EE987A9" Ref="Q28"  Part="2"
 AR Path="/5EEA5FB2/5EE987A9" Ref="Q31"  Part="2"
-F 0 "Q4" H 6244 3746 50  0000 L CNN
+F 0 "Q22" H 6244 3746 50  0000 L CNN
 F 1 "STS8DN6LF6AG" H 6244 3655 50  0000 L CNN
 F 2 "Custom-Footprints:SO-8_3.9x4.9mm_P1.27mm" H 5750 4200 50  0001 C CNN
@@
 	6100 3250 6600 3250
 Text HLabel 5200 2950 0    50   UnSpc ~ 0
-High_ctl_OD
+High_ctl
 Text HLabel 5200 3850 0    50   UnSpc ~ 0
-Low_ctl_OD
+Low_ctl
 Text HLabel 6600 3250 2    50   UnSpc ~ 0
 Low
@@
 	6100 3000 6100 2950
 Text GLabel 6100 2350 1    50   UnSpc ~ 0
-PowerRail
+MatrixPower
 Text Notes 6250 2200 1    50   ~ 0
 5V

Commit message: All traces routed
Changed lines of the file:
@@
 $Descr A 11000 8500
 encoding utf-8
-Sheet 9 14
+Sheet 4 14
 Title "Flip Pixel Board"
 Date "2020-06-20"
@@
 AR Path="/5EEA5FAB/5EE98773" Ref="R19"  Part="1"
 AR Path="/5EEA5FB2/5EE98773" Ref="R21"  Part="1"
-F 0 "R15" H 5500 2600 50  0000 R CNN
+F 0 "R21" H 5500 2600 50  0000 R CNN
 F 1 "R" H 5450 2500 50  0000 R CNN
 F 2 "Resistor_SMD:R_0805_2012Metric" V 5230 2550 50  0001 C CNN
@@
 AR Path="/5EEA5FAB/5EE9878C" Ref="R20"  Part="1"
 AR Path="/5EEA5FB2/5EE9878C" Ref="R22"  Part="1"
-F 0 "R16" H 5500 3550 50  0000 R CNN
+F 0 "R22" H 5500 3550 50  0000 R CNN
 F 1 "R" H 5450 3450 50  0000 R CNN
 F 2 "Resistor_SMD:R_0805_2012Metric" V 5230 3500 50  0001 C CNN
@@
 AR Path="/5EEA5FAB/5EE9879E" Ref="Q28"  Part="1"
 AR Path="/5EEA5FB2/5EE9879E" Ref="Q31"  Part="1"
-F 0 "Q22" H 6244 2796 50  0000 L CNN
+F 0 "Q31" H 6244 2796 50  0000 L CNN
 F 1 "STS8DN6LF6AG" H 6244 2705 50  0000 L CNN
 F 2 "Custom-Footprints:SO-8_3.9x4.9mm_P1.27mm" H 5750 3250 50  0001 C CNN
@@
 AR Path="/5EEA5FAB/5EE987A9" Ref="Q28"  Part="2"
 AR Path="/5EEA5FB2/5EE987A9" Ref="Q31"  Part="2"
-F 0 "Q22" H 6244 3746 50  0000 L CNN
+F 0 "Q31" H 6244 3746 50  0000 L CNN
 F 1 "STS8DN6LF6AG" H 6244 3655 50  0000 L CNN
 F 2 "Custom-Footprints:SO-8_3.9x4.9mm_P1.27mm" H 5750 4200 50  0001 C CNN
