File: microcontroller.sch (KiCad schematic (older format))
At the start: 25 parts, among them Q1 DMN62D0U-7, U5 MCP2221A, U6 ESP32, U7 NPIC6C596ADJ, U8 NPIC6C596ADJ, U9 NPIC6C596ADJ

Commit message: more layout work
Connections:
- net Col1H renamed MatrixControl11
- net Col1L renamed MatrixControl10
- net Col2H renamed MatrixControl20
- net Col2L renamed MatrixControl12
- net Col3H renamed MatrixControl15
- net Col3L renamed MatrixControl14
- net Col4H renamed MatrixControl17
- net Col4L renamed MatrixControl16
- net Col5H renamed MatrixControl19
- net Col5L renamed MatrixControl18
- net Row1H renamed MatrixControl4
- net Row1L renamed MatrixControl3
- net Row2H renamed MatrixControl1
- net Row2L renamed MatrixControl2
- net Row3H renamed MatrixControl5
- net Row3L renamed MatrixControl6
- net Row4H renamed MatrixControl7
- net Row4L renamed MatrixControl13
- net Row5H renamed MatrixControl9
- net Row5L renamed MatrixControl8
Other:
- moved on the sheet: U7, U8, U9

Commit message: All traces routed
Parts:
- added C11, C12, C13, C14, C15: 0.1uF, Capacitor_SMD:C_0805_2012Metric, symbol Device:C
- added TP5, TP6: TestPoint, TestPoint:TestPoint_Pad_D2.0mm, symbol Connector:TestPoint
Connections:
- net scl is gone; now on net SCL: U6.36 (IO22)
- net sda is gone; now on net SDA: U6.37 (IO23)
- net +3V3: now also R26.1, R27.1, R28.1, R29.1, C11.1, C12.1, C13.1, C14.1, C15.1, TP5.1
- net GND: now also C11.2, C12.2, C13.2, C14.2, C15.2, TP6.1
- net IND_SR1_1: now also D55.1; no longer R26.2
- net IND_SR1_2: now also D56.1; no longer R27.2
- net IND_SR2: now also D57.1; no longer R28.2
- net IND_SR3: now also D58.1; no longer R29.2
- net MatrixControl1: now also U8.12 (Q5); no longer U7.6 (Q3)
- net MatrixControl10: now also U9.11 (Q4); no longer U8.11 (Q4)
- net MatrixControl11: now also U8.3 (Q0); no longer U8.12 (Q5)
- net MatrixControl12: now also U8.4 (Q1); no longer U8.13 (Q6)
- net MatrixControl13: now also U8.5 (Q2); no longer U8.3 (Q0)
- net MatrixControl14: now also U8.6 (Q3); no longer U9.5 (Q2)
- net MatrixControl15: now also U7.11 (Q4); no longer U9.6 (Q3)
- net MatrixControl16: now also U7.12 (Q5); no longer U9.11 (Q4)
- net MatrixControl17: now also U7.3 (Q0); no longer U9.12 (Q5)
- net MatrixControl18: now also U7.4 (Q1); no longer U9.13 (Q6)
- net MatrixControl19: now also U7.5 (Q2); no longer U9.14 (Q7)
- net MatrixControl2: now also U8.13 (Q6); no longer U7.5 (Q2)
- net MatrixControl20: now also U7.6 (Q3); no longer U9.4 (Q1)
- net MatrixControl3: now also U8.11 (Q4); no longer U7.3 (Q0)
- net MatrixControl4: now also U9.6 (Q3); no longer U7.4 (Q1)
- net MatrixControl5: now also U9.5 (Q2); no longer U7.12 (Q5)
- net MatrixControl6: now also U9.4 (Q1); no longer U7.11 (Q4)
- net MatrixControl7: now also U9.14 (Q7); no longer U8.4 (Q1)
- net MatrixControl8: now also U9.13 (Q6); no longer U8.5 (Q2)
- net MatrixControl9: now also U9.12 (Q5); no longer U8.6 (Q3)
- net data: now also U6.28 (IO17); no longer U6.30 (IO18)
- net storage_clock: now also U6.30 (IO18); no longer U6.28 (IO17)
- removed net +5V: D55.2, D56.2, D57.2, D58.2
- new net: D55.2, R26.2
- new net: D56.2, R27.2
- new net: D57.2, R28.2
- new net: D58.2, R29.2
Other:
- note added: "Near U5"
- note added: "Near U6"
- note added: "Near U7"
- note added: "Near U8"
- note added: "Near U9"
- moved on the sheet: C10, D55, D56, D57, D58, R26, R27, R28, R29, TP1, TP2, TP3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
