File: power.sch (KiCad schematic (older format))
At the start: 18 parts, among them U1 LM2665M6, U2 TPS79933, U3 ASSR-4118-503E, U4 INA250A3

Commit message: more layout work
Parts:
- JP1: footprint Connector_USB:USB_Micro-AB_Molex_47590-0001 -> Jumper:SolderJumper-2_P1.3mm_Open_RoundedPad1.0x1.5mm
Other:
- note added: "Bypass Cap\nNear U4"
- note added: "Filter Cap\nNear U4"
- note removed: "Bypass Cap\nNear U3"
- note removed: "Filter Cap\nNear U3"
Changed lines of the file:
@@
 F 0 "JP1" H 4200 5850 50  0000 C CNN
 F 1 "BypassJumper" H 4600 5850 50  0000 C CNN
-F 2 "Connector_USB:USB_Micro-AB_Molex_47590-0001" H 4500 5750 50  0001 C CNN
+F 2 "Jumper:SolderJumper-2_P1.3mm_Open_RoundedPad1.0x1.5mm" H 4500 5750 50  0001 C CNN
 F 3 "~" H 4500 5750 50  0001 C CNN
 	1    4500 5750
@@
 current
 Text Notes 750  7450 0    50   ~ 0
-Bypass Cap\nNear U3
+Bypass Cap\nNear U4
 Text Notes 1300 7450 0    50   ~ 0
-Filter Cap\nNear U3
+Filter Cap\nNear U4
 Wire Wire Line
 	900  6750 900  6250

Commit message: All traces routed
Connections:
- net Power_Input is gone; now on net 5V: C1.1
- net 10V: now also D52.2
Changed lines of the file:
@@
 Text Notes 1300 7450 0    50   ~ 0
 Filter Cap\nNear U4
-Wire Wire Line
-	900  6750 900  6250
-Text Label 900  6250 3    50   ~ 0
-Power_Input
 Text HLabel 3650 5950 0    50   Input ~ 0
 5V
@@
 Wire Wire Line
 	5050 1250 5050 1350
+Text HLabel 900  6650 1    50   Input ~ 0
+5V
+Wire Wire Line
+	900  6650 900  6750
+Text HLabel 7950 4850 1    50   Output ~ 0
+10V
 $EndSCHEMATC
