File: flip-pixel.kicad_pcb (KiCad board)
At the start: 2 copper layers, 157.5 x 129.5 mm, 184 parts, among them J1 Barrel-Jack, Q1 DMN62D0U-7, Q10 STS8DN6LF6AG, Q11 DMN62D0U-7, Q12 DMN62D0U-7, Q13 STS8DN6LF6AG, Q14 DMN62D0U-7, Q15 DMN62D0U-7, Q16 STS8DN6LF6AG, Q17 DMN62D0U-7, Q18 DMN62D0U-7, Q19 STS8DN6LF6AG, Q2 DMN62D0U-7, Q20 DMN62D0U-7, Q21 DMN62D0U-7, Q22 STS8DN6LF6AG, Q23 DMN62D0U-7, Q24 DMN62D0U-7, Q25 STS8DN6LF6AG, Q26 DMN62D0U-7, Q27 DMN62D0U-7, Q28 STS8DN6LF6AG, Q29 DMN62D0U-7, Q3 DMN62D0U-7, Q30 DMN62D0U-7, Q31 STS8DN6LF6AG, Q4 STS8DN6LF6AG, Q5 DMN62D0U-7, Q6 DMN62D0U-7, Q7 STS8DN6LF6AG, Q8 DMN62D0U-7, Q9 DMN62D0U-7, U1 LM2665M6, U2 ESP32_DevBoard, U3 INA250A3

Commit message: started work on layout
Parts:
- removed D10, D11, D12, D13, D14, D15, D16, D17, D18, D19, D20, D21, D22, D23, D24, D25, D26, D27, D28, D29, D30, D31, D32, D33, D34, D35, D36, D37, D38, D39, D4, D40, D41, D42, D43, D44, D45, D46, D47, D48, D49, D5, D50, D51, D6, D7, D8, D9: Diode, Diode_SMD:D_SOD-123F
- removed D54, D55, D56, D57, D58, D59, D60, D61, D62, D63, D64, D65, D66, D67, D68, D69, D70, D71, D72, D73: LED_Green, LED_SMD:LED_0805_2012Metric_Pad1.15x1.40mm_HandSolder
- removed Px10, Px11, Px12, Px13, Px14, Px15, Px16, Px17, Px18, Px19, Px2, Px20, Px21, Px22, Px23, Px24, Px25, Px3, Px4, Px5, Px6, Px7, Px8, Px9: FlipPixel, Custom-Footprints:Flip-Pixel
- removed Q11, Q12, Q14, Q15, Q17, Q18, Q2, Q20, Q21, Q23, Q24, Q26, Q27, Q29, Q3, Q30, Q5, Q6, Q8, Q9: DMN62D0U-7, Package_TO_SOT_SMD:SOT-23
- removed R25, R26, R27, R28, R29, R30, R31, R32, R33, R34, R35, R36, R37, R38, R39, R40, R41, R42, R43, R44: R, Resistor_SMD:R_0805_2012Metric
- added C10: 1uF, Capacitor_SMD:C_0805_2012Metric, B.Cu at (252.9, 193.3)
- added C6: C, Capacitor_SMD:C_0805_2012Metric, B.Cu at (286.8, 205.1)
- added C7: C, Capacitor_SMD:C_0805_2012Metric, B.Cu at (286.8, 202.2)
- added C8: C, Capacitor_SMD:C_0805_2012Metric, B.Cu at (286.8, 199.2)
- added C9: 0.1uF, Capacitor_SMD:C_0805_2012Metric, B.Cu at (243.2, 181.4)
- added D2: Diode, Diode_SMD:D_SOD-123F, F.Cu at (181.6, 139.4)
- added D2: Diode, Diode_SMD:D_SOD-123F, F.Cu at (101.6, 119.4)
- added D2: Diode, Diode_SMD:D_SOD-123F, F.Cu at (181.6, 99.4)
- added D2: Diode, Diode_SMD:D_SOD-123F, F.Cu at (161.6, 99.4)
- added D2: Diode, Diode_SMD:D_SOD-123F, F.Cu at (141.6, 99.4)
- added D2: Diode, Diode_SMD:D_SOD-123F, F.Cu at (121.6, 99.4)
- added D2: Diode, Diode_SMD:D_SOD-123F, F.Cu at (101.6, 99.4)
- added D2: Diode, Diode_SMD:D_SOD-123F, F.Cu at (181.6, 79.4)
- added D2: Diode, Diode_SMD:D_SOD-123F, F.Cu at (161.6, 79.4)
- added D2: Diode, Diode_SMD:D_SOD-123F, F.Cu at (141.6, 79.4)
- added D2: Diode, Diode_SMD:D_SOD-123F, F.Cu at (121.6, 79.4)
- added D2: Diode, Diode_SMD:D_SOD-123F, F.Cu at (161.6, 139.4)
- added D2: Diode, Diode_SMD:D_SOD-123F, F.Cu at (101.6, 79.4)
- added D2: Diode, Diode_SMD:D_SOD-123F, F.Cu at (181.6, 59.4)
- added D2: Diode, Diode_SMD:D_SOD-123F, F.Cu at (161.6, 59.4)
- added D2: Diode, Diode_SMD:D_SOD-123F, F.Cu at (141.6, 59.4)
- added D2: Diode, Diode_SMD:D_SOD-123F, F.Cu at (121.6, 59.4)
- added D2: Diode, Diode_SMD:D_SOD-123F, F.Cu at (141.6, 139.4)
- added D2: Diode, Diode_SMD:D_SOD-123F, F.Cu at (121.6, 139.4)
- added D2: Diode, Diode_SMD:D_SOD-123F, F.Cu at (101.6, 139.4)
- added D2: Diode, Diode_SMD:D_SOD-123F, F.Cu at (181.6, 119.4)
- added D2: Diode, Diode_SMD:D_SOD-123F, F.Cu at (161.6, 119.4)
- added D2: Diode, Diode_SMD:D_SOD-123F, F.Cu at (141.6, 119.4)
- added D2: Diode, Diode_SMD:D_SOD-123F, F.Cu at (121.6, 119.4)
- added D3: Diode, Diode_SMD:D_SOD-123F, F.Cu at (181.6, 144.5)
- added D3: Diode, Diode_SMD:D_SOD-123F, F.Cu at (101.6, 124.5)
- added D3: Diode, Diode_SMD:D_SOD-123F, F.Cu at (181.6, 104.5)
- added D3: Diode, Diode_SMD:D_SOD-123F, F.Cu at (161.6, 104.5)
- added D3: Diode, Diode_SMD:D_SOD-123F, F.Cu at (141.6, 104.5)
- added D3: Diode, Diode_SMD:D_SOD-123F, F.Cu at (121.6, 104.5)
- added D3: Diode, Diode_SMD:D_SOD-123F, F.Cu at (101.6, 104.5)
- added D3: Diode, Diode_SMD:D_SOD-123F, F.Cu at (181.6, 84.5)
- added D3: Diode, Diode_SMD:D_SOD-123F, F.Cu at (161.6, 84.5)
- added D3: Diode, Diode_SMD:D_SOD-123F, F.Cu at (141.6, 84.5)
- added D3: Diode, Diode_SMD:D_SOD-123F, F.Cu at (121.6, 84.5)
- added D3: Diode, Diode_SMD:D_SOD-123F, F.Cu at (161.6, 144.5)
- added D3: Diode, Diode_SMD:D_SOD-123F, F.Cu at (101.6, 84.5)
- added D3: Diode, Diode_SMD:D_SOD-123F, F.Cu at (181.6, 64.5)
- added D3: Diode, Diode_SMD:D_SOD-123F, F.Cu at (161.6, 64.5)
- added D3: Diode, Diode_SMD:D_SOD-123F, F.Cu at (141.6, 64.5)
- added D3: Diode, Diode_SMD:D_SOD-123F, F.Cu at (121.6, 64.5)
- added D3: Diode, Diode_SMD:D_SOD-123F, F.Cu at (141.6, 144.5)
- added D3: Diode, Diode_SMD:D_SOD-123F, F.Cu at (121.6, 144.5)
- added D3: Diode, Diode_SMD:D_SOD-123F, F.Cu at (101.6, 144.5)
- added D3: Diode, Diode_SMD:D_SOD-123F, F.Cu at (181.6, 124.5)
- added D3: Diode, Diode_SMD:D_SOD-123F, F.Cu at (161.6, 124.5)
- added D3: Diode, Diode_SMD:D_SOD-123F, F.Cu at (141.6, 124.5)
- added D3: Diode, Diode_SMD:D_SOD-123F, F.Cu at (121.6, 124.5)
- added J2: USB_B_Micro, Connector_USB:USB_Micro-B_Amphenol_10103594-0001LF_Horizontal, B.Cu at (280.5, 190.8)
- added Px1: FlipPixel, Custom-Footprints:Flip-Pixel, F.Cu at (176.3, 141.7)
- added Px1: FlipPixel, Custom-Footprints:Flip-Pixel, F.Cu at (96.3, 121.7)
- added Px1: FlipPixel, Custom-Footprints:Flip-Pixel, F.Cu at (176.3, 101.7)
- added Px1: FlipPixel, Custom-Footprints:Flip-Pixel, F.Cu at (156.3, 101.7)
- added Px1: FlipPixel, Custom-Footprints:Flip-Pixel, F.Cu at (136.3, 101.7)
- added Px1: FlipPixel, Custom-Footprints:Flip-Pixel, F.Cu at (116.3, 101.7)
- added Px1: FlipPixel, Custom-Footprints:Flip-Pixel, F.Cu at (96.3, 101.7)
- added Px1: FlipPixel, Custom-Footprints:Flip-Pixel, F.Cu at (176.3, 81.7)
- added Px1: FlipPixel, Custom-Footprints:Flip-Pixel, F.Cu at (156.3, 81.7)
- added Px1: FlipPixel, Custom-Footprints:Flip-Pixel, F.Cu at (136.3, 81.7)
- added Px1: FlipPixel, Custom-Footprints:Flip-Pixel, F.Cu at (116.3, 81.7)
- added Px1: FlipPixel, Custom-Footprints:Flip-Pixel, F.Cu at (156.3, 141.7)
- added Px1: FlipPixel, Custom-Footprints:Flip-Pixel, F.Cu at (96.3, 81.7)
- added Px1: FlipPixel, Custom-Footprints:Flip-Pixel, F.Cu at (176.3, 61.7)
- added Px1: FlipPixel, Custom-Footprints:Flip-Pixel, F.Cu at (156.3, 61.7)
- added Px1: FlipPixel, Custom-Footprints:Flip-Pixel, F.Cu at (136.3, 61.7)
- added Px1: FlipPixel, Custom-Footprints:Flip-Pixel, F.Cu at (116.3, 61.7)
- added Px1: FlipPixel, Custom-Footprints:Flip-Pixel, F.Cu at (136.3, 141.7)
- added Px1: FlipPixel, Custom-Footprints:Flip-Pixel, F.Cu at (116.3, 141.7)
- added Px1: FlipPixel, Custom-Footprints:Flip-Pixel, F.Cu at (96.3, 141.7)
- added Px1: FlipPixel, Custom-Footprints:Flip-Pixel, F.Cu at (176.3, 121.7)
- added Px1: FlipPixel, Custom-Footprints:Flip-Pixel, F.Cu at (156.3, 121.7)
- added Px1: FlipPixel, Custom-Footprints:Flip-Pixel, F.Cu at (136.3, 121.7)
- added Px1: FlipPixel, Custom-Footprints:Flip-Pixel, F.Cu at (116.3, 121.7)
- added TP1: TestPoint, TestPoint:TestPoint_Pad_D2.0mm, B.Cu at (262.3, 198.0)
- added TP2: TestPoint, TestPoint:TestPoint_Pad_D2.0mm, B.Cu at (252.7, 189.8)
- added TP3: TestPoint, TestPoint:TestPoint_Pad_D2.0mm, B.Cu at (257.1, 192.7)
- added TP4: TestPoint, TestPoint:TestPoint_Pad_D2.0mm, B.Cu at (247.4, 180.9)
- added U4: INA250A3, Package_SO:TSSOP-16_4.4x5mm_P0.65mm, B.Cu at (280.2, 203.3)
- added U5: MCP2221A, Package_SO:TSSOP-14_4.4x5mm_P0.65mm, B.Cu at (264.7, 203.3)
- added U6: ESP32, Custom-Footprints:MODULE_ESP32-WROOM-32, F.Cu at (67.3, 124.5)
- added U7: NPIC6C596ADJ, Package_SO:SOIC-16_4.55x10.3mm_P1.27mm, B.Cu at (132.8, 92.8)
- added U8: NPIC6C596ADJ, Package_SO:SOIC-16_4.55x10.3mm_P1.27mm, B.Cu at (142.9, 93.1)
- added U9: NPIC6C596ADJ, Package_SO:SOIC-16_4.55x10.3mm_P1.27mm, B.Cu at (153.3, 93.0)
- C1: value C -> 0.1uF
- C4: value 0.1uF -> C
- D2, D3: moved to F.Cu
- JP1: footprint Jumper:SolderJumper-2_P1.3mm_Open_RoundedPad1.0x1.5mm -> Connector_USB:USB_Micro-AB_Molex_47590-0001
- Q10, Q13, Q16, Q19, Q22, Q25, Q28, Q31, Q4, Q7: moved to B.Cu
- U2: value ESP32_DevBoard -> TPS79933; footprint Custom-Footprints:DIP-38_900_ELL -> Package_TO_SOT_SMD:SOT-23-5
- U3: value INA250A3 -> ASSR-4118-503E; footprint Package_SO:TSSOP-16_4.4x5mm_P0.65mm -> Package_SO:SO-4_4.4x4.3mm_P2.54mm
- moved Q31 84.3 mm to (90.3, 55.8)
- moved Q22 79.5 mm to (171.6, 55.8)
- moved C3 50.8 mm to (17.7, 88.6)
- moved C4 50.8 mm to (20.2, 74.3)
- moved Q1 50.8 mm to (18.7, 94.6)
- moved R1 50.8 mm to (18.7, 91.6)
- moved R2 50.8 mm to (19.7, 88.6)
- moved C2 50.8 mm to (14.4, 91.6)
- moved D1 50.8 mm to (14.4, 85.4)
- moved D52 50.8 mm to (21.9, 94.7)
- moved U1 50.8 mm to (14.4, 88.5)
- moved C1 50.8 mm to (10.8, 88.5)
- moved C5 50.8 mm to (15.0, 78.5)
- moved D53 50.8 mm to (21.9, 88.6)
- moved R23 50.8 mm to (21.9, 94.7)
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Connections:
- net /Column1/Gate_H renamed /Column1/High_ctl_OD
- net /Column1/Gate_L renamed /Column1/Low_ctl_OD
- net /Column2/Gate_H renamed /Column2/High_ctl_OD
- net /Column2/Gate_L renamed /Column2/Low_ctl_OD
- net /Column3/Gate_H renamed /Column3/High_ctl_OD
- net /Column3/Gate_L renamed /Column3/Low_ctl_OD
- net /Column4/Gate_H renamed /Column4/High_ctl_OD
- net /Column4/Gate_L renamed /Column4/Low_ctl_OD
- net /Column5/Gate_H renamed /Column5/High_ctl_OD
- net /Column5/Gate_L renamed /Column5/Low_ctl_OD
- net /Row1/Gate_H renamed /Row1/High_ctl_OD
- net /Row1/Gate_L renamed /Row1/Low_ctl_OD
- net /Row2/Gate_H renamed /Row2/High_ctl_OD
- net /Row2/Gate_L renamed /Row2/Low_ctl_OD
- net /Row3/Gate_H renamed /Row3/High_ctl_OD
- net /Row3/Gate_L renamed /Row3/Low_ctl_OD
- net /Row4/Gate_H renamed /Row4/High_ctl_OD
- net /Row4/Gate_L renamed /Row4/Low_ctl_OD
- net /Row5/Gate_H renamed /Row5/High_ctl_OD
- net /Row5/Gate_L renamed /Row5/Low_ctl_OD
- C1 pad 1: +5V -> /Power/Power_Input
- C2 pad 1: Net-(C2-Pad1) -> /Power/matrix_current
- C2 pad 2: Net-(C2-Pad2) -> GND
- C3 pad 1: +10V -> +5V
- C4 pad 1: /Power_Input -> Net-(C4-Pad1)
- C4 pad 2: GND -> Net-(C4-Pad2)
- C5 pad 1: /current -> +5V
- D1 pad 1: +10V -> Net-(C6-Pad1)
- D52 pad 2: /shutdown -> Net-(D52-Pad2)
- D53 pad 2: +10V -> /Controller/usb_indicator
- J1 pad 1: /Power_Input -> +5V
- JP1 pad 1: /Power_Input -> +5V
- JP1 pad 2: +5V -> MatrixPower
- Q1 pad 1: /enable -> /Controller/esp_reset
- Q1 pad 3: /shutdown -> /Controller/~esp_reset
- Q10 pad 7: +5V -> PowerRail
- Q10 pad 8: +5V -> PowerRail
- Q13 pad 7: +5V -> PowerRail
- Q13 pad 8: +5V -> PowerRail
- Q16 pad 7: +5V -> PowerRail
- Q16 pad 8: +5V -> PowerRail
- Q19 pad 7: +5V -> PowerRail
- Q19 pad 8: +5V -> PowerRail
- Q22 pad 7: +5V -> PowerRail
- Q22 pad 8: +5V -> PowerRail
- Q25 pad 7: +5V -> PowerRail
- Q25 pad 8: +5V -> PowerRail
- Q28 pad 7: +5V -> PowerRail
- Q28 pad 8: +5V -> PowerRail
- Q31 pad 7: +5V -> PowerRail
- Q31 pad 8: +5V -> PowerRail
- Q4 pad 7: +5V -> PowerRail
- Q4 pad 8: +5V -> PowerRail
- Q7 pad 7: +5V -> PowerRail
- Q7 pad 8: +5V -> PowerRail
- R1 pad 1: +5V -> Net-(R1-Pad1)
- R1 pad 2: /shutdown -> GND
- R10 pad 1: +10V -> /GateDrive
- R11 pad 1: +10V -> /GateDrive
- R12 pad 1: +10V -> /GateDrive
- R13 pad 1: +10V -> /GateDrive
- R14 pad 1: +10V -> /GateDrive
- R15 pad 1: +10V -> /GateDrive
- R16 pad 1: +10V -> /GateDrive
- R17 pad 1: +10V -> /GateDrive
- R18 pad 1: +10V -> /GateDrive
- R19 pad 1: +10V -> /GateDrive
- R2 pad 1: +10V -> /GateDrive
- R20 pad 1: +10V -> /GateDrive
- R21 pad 1: +10V -> /GateDrive
- R22 pad 1: +10V -> /GateDrive
- R3 pad 1: +10V -> /GateDrive
- R4 pad 1: +10V -> /GateDrive
- R5 pad 1: +10V -> /GateDrive
- R6 pad 1: +10V -> /GateDrive
- R7 pad 1: +10V -> /GateDrive
- R8 pad 1: +10V -> /GateDrive
- R9 pad 1: +10V -> /GateDrive
- U1 pad 3: Net-(C2-Pad2) -> Net-(C4-Pad2)
- U1 pad 4: /shutdown -> GND
- U1 pad 5: +10V -> Net-(C6-Pad1)
- U1 pad 6: Net-(C2-Pad1) -> Net-(C4-Pad1)
- U2 pad 1: Net-(U2-Pad1) -> +5V
- U2 pad 2: Net-(U2-Pad2) -> GND
- U2 pad 3: Net-(U2-Pad3) -> +5V
- U2 pad 4: /current -> Net-(C7-Pad1)
- U2 pad 5: /Col5H -> +3V3
- U3 pad 1: +5V -> /Power/10V_enable
- U3 pad 2: +5V -> Net-(R1-Pad1)
- U3 pad 3: +5V -> /GateDrive
- U3 pad 4: Net-(U3-Pad4) -> Net-(C6-Pad1)
Routing:
- net /Row1/High: track 108.3 -> 528.2 mm
- net /Row1/Low: track 104.8 -> 505.6 mm
- net /Row5H: track 340.3 -> 0.00 mm, vias 2 -> 0
- net /Row5L: track 331.7 -> 0.00 mm, vias 2 -> 0
- net /Row4H: track 318.2 -> 0.00 mm, vias 2 -> 0
- net +10V: track 313.1 -> 0.00 mm, vias 25 -> 0
- net /Row4L: track 310.7 -> 0.00 mm, vias 2 -> 0
- net /Row3H: track 297.2 -> 0.00 mm, vias 2 -> 0
- net /Row3L: track 289.8 -> 0.00 mm, vias 2 -> 0
- net /Row2H: track 278.9 -> 0.00 mm, vias 2 -> 0
- net /Row2L: track 274.0 -> 0.00 mm, vias 2 -> 0
- net /Row1H: track 266.3 -> 0.00 mm, vias 2 -> 0
- net /Row1L: track 258.9 -> 0.00 mm, vias 2 -> 0
- net /Col5H: track 199.1 -> 0.00 mm
- net /Col5L: track 188.4 -> 0.00 mm
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- removed copper zone on B.Cu, net +5V
- removed copper zone on F.Cu, net +5V
- removed copper zone on F.Cu, net /PixelMatrix/Col_1
- removed copper zone on F.Cu, net /PixelMatrix/Col_2
- removed copper zone on F.Cu, net /PixelMatrix/Col_3
- removed copper zone on F.Cu, net /PixelMatrix/Col_4
- removed copper zone on F.Cu, net /PixelMatrix/Col_5
- removed copper zone on F.Cu, net /Power_Input
- removed copper zone on F.Cu, net /Row1/High
- removed copper zone on F.Cu, net /Row2/High
- removed copper zone on F.Cu, net /Row3/High
- removed copper zone on F.Cu, net /Row4/High
- removed copper zone on F.Cu, net /Row5/High
- removed copper zone on B.Cu, net GND
- removed copper zone on F.Cu, net GND
Other:
- board size 157.5 x 129.5 mm -> 157.6 x 129.5 mm
- board text removed: "H"
- board text removed: "L"

Commit message: more layout work
Parts:
- removed the C4 at (20.2, 74.3)
- removed the D2 at (181.6, 139.4)
- removed the D2 at (101.6, 119.4)
- removed the D2 at (181.6, 99.4)
- removed the D2 at (161.6, 99.4)
- removed the D2 at (141.6, 99.4)
- removed the D2 at (121.6, 99.4)
- removed the D2 at (101.6, 99.4)
- removed the D2 at (181.6, 79.4)
- removed the D2 at (161.6, 79.4)
- removed the D2 at (141.6, 79.4)
- removed the D2 at (121.6, 79.4)
- removed the D2 at (161.6, 139.4)
- removed the D2 at (101.6, 79.4)
- removed the D2 at (181.6, 59.4)
- removed the D2 at (161.6, 59.4)
- removed the D2 at (141.6, 59.4)
- removed the D2 at (121.6, 59.4)
- removed the D2 at (141.6, 139.4)
- removed the D2 at (121.6, 139.4)
- removed the D2 at (101.6, 139.4)
- removed the D2 at (181.6, 119.4)
- removed the D2 at (161.6, 119.4)
- removed the D2 at (141.6, 119.4)
- removed the D2 at (121.6, 119.4)
- removed the D3 at (181.6, 144.5)
- removed the D3 at (101.6, 124.5)
- removed the D3 at (181.6, 104.5)
- removed the D3 at (161.6, 104.5)
- removed the D3 at (141.6, 104.5)
- removed the D3 at (121.6, 104.5)
- removed the D3 at (101.6, 104.5)
- removed the D3 at (181.6, 84.5)
- removed the D3 at (161.6, 84.5)
- removed the D3 at (141.6, 84.5)
- removed the D3 at (121.6, 84.5)
- removed the D3 at (161.6, 144.5)
- removed the D3 at (101.6, 84.5)
- removed the D3 at (181.6, 64.5)
- removed the D3 at (161.6, 64.5)
- removed the D3 at (141.6, 64.5)
- removed the D3 at (121.6, 64.5)
- removed the D3 at (141.6, 144.5)
- removed the D3 at (121.6, 144.5)
- removed the D3 at (101.6, 144.5)
- removed the D3 at (181.6, 124.5)
- removed the D3 at (161.6, 124.5)
- removed the D3 at (141.6, 124.5)
- removed the D3 at (121.6, 124.5)
- removed the Px1 at (176.3, 141.7)
- removed the Px1 at (96.3, 121.7)
- removed the Px1 at (176.3, 101.7)
- removed the Px1 at (156.3, 101.7)
- removed the Px1 at (136.3, 101.7)
- removed the Px1 at (116.3, 101.7)
- removed the Px1 at (96.3, 101.7)
- removed the Px1 at (176.3, 81.7)
- removed the Px1 at (156.3, 81.7)
- removed the Px1 at (136.3, 81.7)
- removed the Px1 at (116.3, 81.7)
- removed the Px1 at (156.3, 141.7)
- removed the Px1 at (96.3, 81.7)
- removed the Px1 at (136.3, 141.7)
- removed the Px1 at (116.3, 141.7)
- removed the Px1 at (96.3, 141.7)
- removed the Px1 at (176.3, 121.7)
- removed the Px1 at (156.3, 121.7)
- removed the Px1 at (136.3, 121.7)
- removed the Px1 at (116.3, 121.7)
- added C2: C, Capacitor_SMD:C_0805_2012Metric, F.Cu at (57.4, 63.4)
- added D2: Diode, Diode_SMD:D_SOD-123F, F.Cu at (182.0, 138.5)
- added D2: Diode, Diode_SMD:D_SOD-123F, F.Cu at (102.0, 118.5)
- added D2: Diode, Diode_SMD:D_SOD-123F, F.Cu at (182.0, 98.5)
- added D2: Diode, Diode_SMD:D_SOD-123F, F.Cu at (162.0, 98.5)
- added D2: Diode, Diode_SMD:D_SOD-123F, F.Cu at (142.0, 98.5)
- added D2: Diode, Diode_SMD:D_SOD-123F, F.Cu at (122.0, 98.5)
- added D2: Diode, Diode_SMD:D_SOD-123F, F.Cu at (102.0, 98.5)
- added D2: Diode, Diode_SMD:D_SOD-123F, F.Cu at (182.0, 78.5)
- added D2: Diode, Diode_SMD:D_SOD-123F, F.Cu at (162.0, 78.5)
- added D2: Diode, Diode_SMD:D_SOD-123F, F.Cu at (142.0, 78.5)
- added D2: Diode, Diode_SMD:D_SOD-123F, F.Cu at (122.0, 78.5)
- added D2: Diode, Diode_SMD:D_SOD-123F, F.Cu at (162.0, 138.5)
- added D2: Diode, Diode_SMD:D_SOD-123F, F.Cu at (102.0, 78.5)
- added D2: Diode, Diode_SMD:D_SOD-123F, F.Cu at (182.0, 58.5)
- added D2: Diode, Diode_SMD:D_SOD-123F, F.Cu at (162.0, 58.5)
- added D2: Diode, Diode_SMD:D_SOD-123F, F.Cu at (142.0, 58.5)
- added D2: Diode, Diode_SMD:D_SOD-123F, F.Cu at (122.0, 58.5)
- added D2: Diode, Diode_SMD:D_SOD-123F, F.Cu at (142.0, 138.5)
- added D2: Diode, Diode_SMD:D_SOD-123F, F.Cu at (122.0, 138.5)
- added D2: Diode, Diode_SMD:D_SOD-123F, F.Cu at (102.0, 138.5)
- added D2: Diode, Diode_SMD:D_SOD-123F, F.Cu at (182.0, 118.5)
- added D2: Diode, Diode_SMD:D_SOD-123F, F.Cu at (162.0, 118.5)
- added D2: Diode, Diode_SMD:D_SOD-123F, F.Cu at (142.0, 118.5)
- added D2: Diode, Diode_SMD:D_SOD-123F, F.Cu at (122.0, 118.5)
- added D3: Diode, Diode_SMD:D_SOD-123F, F.Cu at (182.0, 143.5)
- added D3: Diode, Diode_SMD:D_SOD-123F, F.Cu at (102.0, 123.5)
- added D3: Diode, Diode_SMD:D_SOD-123F, F.Cu at (182.0, 103.5)
- added D3: Diode, Diode_SMD:D_SOD-123F, F.Cu at (162.0, 103.5)
- added D3: Diode, Diode_SMD:D_SOD-123F, F.Cu at (142.0, 103.5)
- added D3: Diode, Diode_SMD:D_SOD-123F, F.Cu at (122.0, 103.5)
- added D3: Diode, Diode_SMD:D_SOD-123F, F.Cu at (102.0, 103.5)
- added D3: Diode, Diode_SMD:D_SOD-123F, F.Cu at (182.0, 83.5)
- added D3: Diode, Diode_SMD:D_SOD-123F, F.Cu at (162.0, 83.5)
- added D3: Diode, Diode_SMD:D_SOD-123F, F.Cu at (142.0, 83.5)
- added D3: Diode, Diode_SMD:D_SOD-123F, F.Cu at (122.0, 83.5)
- added D3: Diode, Diode_SMD:D_SOD-123F, F.Cu at (162.0, 143.5)
- added D3: Diode, Diode_SMD:D_SOD-123F, F.Cu at (102.0, 83.5)
- added D3: Diode, Diode_SMD:D_SOD-123F, F.Cu at (182.0, 63.5)
- added D3: Diode, Diode_SMD:D_SOD-123F, F.Cu at (162.0, 63.5)
- added D3: Diode, Diode_SMD:D_SOD-123F, F.Cu at (142.0, 63.5)
- added D3: Diode, Diode_SMD:D_SOD-123F, F.Cu at (122.0, 63.5)
- added D3: Diode, Diode_SMD:D_SOD-123F, F.Cu at (142.0, 143.5)
- added D3: Diode, Diode_SMD:D_SOD-123F, F.Cu at (122.0, 143.5)
- added D3: Diode, Diode_SMD:D_SOD-123F, F.Cu at (102.0, 143.5)
- added D3: Diode, Diode_SMD:D_SOD-123F, F.Cu at (182.0, 123.5)
- added D3: Diode, Diode_SMD:D_SOD-123F, F.Cu at (162.0, 123.5)
- added D3: Diode, Diode_SMD:D_SOD-123F, F.Cu at (142.0, 123.5)
- added D3: Diode, Diode_SMD:D_SOD-123F, F.Cu at (122.0, 123.5)
- added D54: LED_Green, LED_SMD:LED_0805_2012Metric_Pad1.15x1.40mm_HandSolder, F.Cu at (74.0, 138.0)
- added D55: LED_Green, LED_SMD:LED_0805_2012Metric_Pad1.15x1.40mm_HandSolder, F.Cu at (47.5, 85.5)
- added D56: LED_Green, LED_SMD:LED_0805_2012Metric_Pad1.15x1.40mm_HandSolder, F.Cu at (47.5, 83.5)
- added D57: LED_Green, LED_SMD:LED_0805_2012Metric_Pad1.15x1.40mm_HandSolder, F.Cu at (47.5, 80.5)
- added D58: LED_Green, LED_SMD:LED_0805_2012Metric_Pad1.15x1.40mm_HandSolder, F.Cu at (47.5, 78.5)
- added Px1: FlipPixel, Custom-Footprints:Flip-Pixel, F.Cu at (96.0, 141.0)
- added Px1: FlipPixel, Custom-Footprints:Flip-Pixel, F.Cu at (96.0, 121.0)
- added Px1: FlipPixel, Custom-Footprints:Flip-Pixel, F.Cu at (96.0, 101.0)
- added Px1: FlipPixel, Custom-Footprints:Flip-Pixel, F.Cu at (96.0, 81.0)
- added Px11: FlipPixel, Custom-Footprints:Flip-Pixel, F.Cu at (136.0, 141.0)
- added Px11: FlipPixel, Custom-Footprints:Flip-Pixel, F.Cu at (136.0, 121.0)
- added Px11: FlipPixel, Custom-Footprints:Flip-Pixel, F.Cu at (136.0, 101.0)
- added Px11: FlipPixel, Custom-Footprints:Flip-Pixel, F.Cu at (136.0, 81.0)
- added Px16: FlipPixel, Custom-Footprints:Flip-Pixel, F.Cu at (156.0, 141.0)
- added Px16: FlipPixel, Custom-Footprints:Flip-Pixel, F.Cu at (156.0, 121.0)
- added Px16: FlipPixel, Custom-Footprints:Flip-Pixel, F.Cu at (156.0, 101.0)
- added Px16: FlipPixel, Custom-Footprints:Flip-Pixel, F.Cu at (156.0, 81.0)
- added Px21: FlipPixel, Custom-Footprints:Flip-Pixel, F.Cu at (176.0, 141.0)
- added Px21: FlipPixel, Custom-Footprints:Flip-Pixel, F.Cu at (176.0, 121.0)
- added Px21: FlipPixel, Custom-Footprints:Flip-Pixel, F.Cu at (176.0, 101.0)
- added Px21: FlipPixel, Custom-Footprints:Flip-Pixel, F.Cu at (176.0, 81.0)
- added Px6: FlipPixel, Custom-Footprints:Flip-Pixel, F.Cu at (116.0, 141.0)
- added Px6: FlipPixel, Custom-Footprints:Flip-Pixel, F.Cu at (116.0, 121.0)
- added Px6: FlipPixel, Custom-Footprints:Flip-Pixel, F.Cu at (116.0, 101.0)
- added Px6: FlipPixel, Custom-Footprints:Flip-Pixel, F.Cu at (116.0, 81.0)
- added R25: R, Resistor_SMD:R_0805_2012Metric, B.Cu at (74.0, 138.0)
- added R26: R, Resistor_SMD:R_0805_2012Metric, B.Cu at (47.5, 85.5)
- added R27: R, Resistor_SMD:R_0805_2012Metric, B.Cu at (47.5, 83.5)
- added R28: R, Resistor_SMD:R_0805_2012Metric, B.Cu at (47.5, 80.5)
- added R29: R, Resistor_SMD:R_0805_2012Metric, B.Cu at (47.5, 78.5)
- added R30: 10k, Resistor_SMD:R_0805_2012Metric, B.Cu at (34.0, 114.4)
- C1: renamed from C6; value C -> 0.1uF; moved to F.Cu
- C3: renamed from C1; value 0.1uF -> C
- C7, C8, C9, J2, Q10, Q13, Q16, Q4, Q7, U4, U5, U7, U8, U9: moved to F.Cu
- JP1: footprint Connector_USB:USB_Micro-AB_Molex_47590-0001 -> Jumper:SolderJumper-2_P1.3mm_Open_RoundedPad1.0x1.5mm
- R10, R11, R12, R13, R14, R15, R16, R17, R18, R19, R20, R21, R22, R3, R4, R5, R6, R7, R8, R9: moved to B.Cu
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- renumbered C2 to C4, C3 to C6, Px1 to Px11, Px1 to Px16, Px1 to Px21, Px1 to Px6
Connections:
- C1 pad 1: Net-(C6-Pad1) -> /Power/Power_Input
- C3 pad 1: /Power/Power_Input -> +5V
- C4 pad 1: /Power/matrix_current -> Net-(C4-Pad1)
- C4 pad 2: GND -> Net-(C4-Pad2)
- C6 pad 1: +5V -> Net-(C6-Pad1)
- Px11 pad 1: Net-(D2-Pad1) -> Net-(D22-Pad1)
- Px11 pad 2: /PixelMatrix/Col_1 -> /PixelMatrix/Col_3
- Px16 pad 1: Net-(D2-Pad1) -> Net-(D32-Pad1)
- Px16 pad 2: /PixelMatrix/Col_1 -> /PixelMatrix/Col_4
- Px21 pad 1: Net-(D2-Pad1) -> Net-(D42-Pad1)
- Px21 pad 2: /PixelMatrix/Col_1 -> /PixelMatrix/Col_5
- Px6 pad 1: Net-(D2-Pad1) -> Net-(D12-Pad1)
- Px6 pad 2: /PixelMatrix/Col_1 -> /PixelMatrix/Col_2
- Q10 pad 2: /Row3/High_ctl_OD -> MatrixControl15
- Q10 pad 4: /Row3/Low_ctl_OD -> MatrixControl16
- Q10 pad 7: PowerRail -> MatrixPower
- Q10 pad 8: PowerRail -> MatrixPower
- Q13 pad 2: /Row4/High_ctl_OD -> MatrixControl17
- Q13 pad 4: /Row4/Low_ctl_OD -> MatrixControl18
- Q13 pad 7: PowerRail -> MatrixPower
- Q13 pad 8: PowerRail -> MatrixPower
- Q16 pad 2: /Row5/High_ctl_OD -> MatrixControl19
- Q16 pad 4: /Row5/Low_ctl_OD -> MatrixControl20
- Q16 pad 7: PowerRail -> MatrixPower
- Q16 pad 8: PowerRail -> MatrixPower
- Q19 pad 2: /Column2/High_ctl_OD -> MatrixControl3
- Q19 pad 4: /Column2/Low_ctl_OD -> MatrixControl4
- Q19 pad 7: PowerRail -> MatrixPower
- Q19 pad 8: PowerRail -> MatrixPower
- Q22 pad 2: /Column1/High_ctl_OD -> MatrixControl1
- Q22 pad 4: /Column1/Low_ctl_OD -> MatrixControl2
- Q22 pad 7: PowerRail -> MatrixPower
- Q22 pad 8: PowerRail -> MatrixPower
- Q25 pad 2: /Column3/High_ctl_OD -> MatrixControl5
- Q25 pad 4: /Column3/Low_ctl_OD -> MatrixControl6
- Q25 pad 7: PowerRail -> MatrixPower
- Q25 pad 8: PowerRail -> MatrixPower
- Q28 pad 2: /Column4/High_ctl_OD -> MatrixControl7
- Q28 pad 4: /Column4/Low_ctl_OD -> MatrixControl8
- Q28 pad 7: PowerRail -> MatrixPower
- Q28 pad 8: PowerRail -> MatrixPower
- Q31 pad 2: /Column5/High_ctl_OD -> MatrixControl9
- Q31 pad 4: /Column5/Low_ctl_OD -> MatrixControl10
- Q31 pad 7: PowerRail -> MatrixPower
- Q31 pad 8: PowerRail -> MatrixPower
- Q4 pad 2: /Row2/High_ctl_OD -> MatrixControl13
- Q4 pad 4: /Row2/Low_ctl_OD -> MatrixControl14
- Q4 pad 7: PowerRail -> MatrixPower
- Q4 pad 8: PowerRail -> MatrixPower
- Q7 pad 2: /Row1/High_ctl_OD -> MatrixControl11
- Q7 pad 4: /Row1/Low_ctl_OD -> MatrixControl12
- Q7 pad 7: PowerRail -> MatrixPower
- Q7 pad 8: PowerRail -> MatrixPower
- R10 pad 2: /Row4/Low_ctl_OD -> MatrixControl18
- R11 pad 2: /Row5/High_ctl_OD -> MatrixControl19
- R12 pad 2: /Row5/Low_ctl_OD -> MatrixControl20
- R13 pad 2: /Column2/High_ctl_OD -> MatrixControl3
- R14 pad 2: /Column2/Low_ctl_OD -> MatrixControl4
- R15 pad 2: /Column1/High_ctl_OD -> MatrixControl1
- R16 pad 2: /Column1/Low_ctl_OD -> MatrixControl2
- R17 pad 2: /Column3/High_ctl_OD -> MatrixControl5
- R18 pad 2: /Column3/Low_ctl_OD -> MatrixControl6
- R19 pad 2: /Column4/High_ctl_OD -> MatrixControl7
- R20 pad 2: /Column4/Low_ctl_OD -> MatrixControl8
- R21 pad 2: /Column5/High_ctl_OD -> MatrixControl9
- R22 pad 2: /Column5/Low_ctl_OD -> MatrixControl10
- R3 pad 2: /Row2/High_ctl_OD -> MatrixControl13
- R4 pad 2: /Row2/Low_ctl_OD -> MatrixControl14
- R5 pad 2: /Row1/High_ctl_OD -> MatrixControl11
- R6 pad 2: /Row1/Low_ctl_OD -> MatrixControl12
- R7 pad 2: /Row3/High_ctl_OD -> MatrixControl15
- R8 pad 2: /Row3/Low_ctl_OD -> MatrixControl16
- R9 pad 2: /Row4/High_ctl_OD -> MatrixControl17
- U7 pad 11: /Controller/Row3L -> MatrixControl6
- U7 pad 12: /Controller/Row3H -> MatrixControl5
- U7 pad 3: /Controller/Row1L -> MatrixControl3
- U7 pad 4: /Controller/Row1H -> MatrixControl4
- U7 pad 5: /Controller/Row2L -> MatrixControl2
- U7 pad 6: /Controller/Row2H -> MatrixControl1
- U8 pad 11: /Controller/Col1L -> MatrixControl10
- U8 pad 12: /Controller/Col1H -> MatrixControl11
- U8 pad 13: /Controller/Col2L -> MatrixControl12
- U8 pad 3: /Controller/Row4L -> MatrixControl13
- U8 pad 4: /Controller/Row4H -> MatrixControl7
- U8 pad 5: /Controller/Row5L -> MatrixControl8
- U8 pad 6: /Controller/Row5H -> MatrixControl9
- U9 pad 11: /Controller/Col4L -> MatrixControl16
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Routing:
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- added copper zone on F.Cu, net /Row1/High
- added copper zone on B.Cu, net GND
- added copper zone on F.Cu, net GND
- added copper zone on F.Cu, net MatrixPower
- removed copper zone on B.Cu, net /PixelMatrix/Col_1
- removed copper zone on B.Cu, net /PixelMatrix/Col_2
- removed copper zone on B.Cu, net /PixelMatrix/Col_3
- removed copper zone on B.Cu, net /PixelMatrix/Col_4
- removed copper zone on B.Cu, net /PixelMatrix/Col_5
- removed copper zone on F.Cu, net /Row2/Low
- removed copper zone on F.Cu, net /Row3/Low
- removed copper zone on F.Cu, net /Row4/Low
- removed copper zone on F.Cu, net /Row5/Low
Other:
- board size 157.6 x 129.5 mm -> 151.4 x 100.4 mm

Commit message: All traces routed
Parts:
- added C11: 0.1uF, Capacitor_SMD:C_0805_2012Metric, B.Cu at (48.1, 135.2)
- added C12: 0.1uF, Capacitor_SMD:C_0805_2012Metric, B.Cu at (43.5, 122.8)
- added C13: 0.1uF, Capacitor_SMD:C_0805_2012Metric, B.Cu at (47.9, 96.0)
- added C14: 0.1uF, Capacitor_SMD:C_0805_2012Metric, B.Cu at (47.9, 86.0)
- added C15: 0.1uF, Capacitor_SMD:C_0805_2012Metric, B.Cu at (47.9, 75.8)
- C1, C2: moved to B.Cu
- J2: value USB_B_Micro -> MicroUSB; footprint Connector_USB:USB_Micro-B_Amphenol_10103594-0001LF_Horizontal -> Custom-Footprints:USB_Micro-B_Amphenol_10104110_Horizontal
- moved JP1 97.9 mm to (77.4, 150.0)
- moved C1 88.8 mm to (75.2, 146.8), turned to 0 degrees
- moved J1 88.7 mm to (49.0, 145.0)
- moved U4 88.3 mm to (77.4, 145.1), turned to 180 degrees
- moved LOGO1 82.7 mm to (46.2, 55.8)
- moved C2 81.8 mm to (75.3, 143.3), turned to 0 degrees
- moved C5 73.5 mm to (57.4, 142.4), turned to 0 degrees
- moved U2 69.2 mm to (57.5, 139.3), turned to 90 degrees
- moved C7 65.0 mm to (57.5, 136.2), turned to 0 degrees
- moved C8 62.2 mm to (57.5, 134.1), turned to 0 degrees
- moved TP1 43.6 mm to (19.0, 157.8)
- moved TP2 43.6 mm to (19.0, 153.8)
- moved TP3 43.6 mm to (15.0, 157.8)
- moved TP4 43.6 mm to (15.0, 153.8)
- moved U5 33.8 mm to (48.2, 132.0)
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- renumbered D2 to D10, D3 to D11, D2 to D12, D3 to D13, D2 to D14, D3 to D15, D2 to D16, D3 to D17, D2 to D18, D3 to D19, D2 to D20, D3 to D21, D2 to D22, D3 to D23, D2 to D24, D3 to D25, D2 to D26, D3 to D27, D2 to D28, D3 to D29, D2 to D30, D3 to D31, D2 to D32, D3 to D33, D2 to D34, D3 to D35, D2 to D36, D3 to D37, D2 to D38, D3 to D39, D2 to D4, D2 to D40, D3 to D41, D2 to D42, D3 to D43, D2 to D44, D3 to D45, D2 to D46, D3 to D47, D2 to D48, D3 to D49, D3 to D5, D2 to D50, D3 to D51, D2 to D6, D3 to D7, D2 to D8, D3 to D9, Px6 to Px10, Px11 to Px12, Px11 to Px13, Px11 to Px14, Px11 to Px15, Px16 to Px17, Px16 to Px18, Px16 to Px19, Px1 to Px2, Px16 to Px20, Px21 to Px22, Px21 to Px23, Px21 to Px24, Px21 to Px25, Px1 to Px3, Px1 to Px4, Px1 to Px5, Px6 to Px7, Px6 to Px8, Px6 to Px9
Connections:
- C1 pad 1: /Power/Power_Input -> +5V
- D10 pad 1: Net-(D2-Pad1) -> Net-(D10-Pad1)
- D10 pad 2: /Row1/High -> /Row5/High
- D11 pad 1: /Row1/Low -> /Row5/Low
- D11 pad 2: Net-(D2-Pad1) -> Net-(D10-Pad1)
- D12 pad 1: Net-(D2-Pad1) -> Net-(D12-Pad1)
- D13 pad 2: Net-(D2-Pad1) -> Net-(D12-Pad1)
- D14 pad 1: Net-(D2-Pad1) -> Net-(D14-Pad1)
- D14 pad 2: /Row1/High -> /Row2/High
- D15 pad 1: /Row1/Low -> /Row2/Low
- D15 pad 2: Net-(D2-Pad1) -> Net-(D14-Pad1)
- D16 pad 1: Net-(D2-Pad1) -> Net-(D16-Pad1)
- D16 pad 2: /Row1/High -> /Row3/High
- D17 pad 1: /Row1/Low -> /Row3/Low
- D17 pad 2: Net-(D2-Pad1) -> Net-(D16-Pad1)
- D18 pad 1: Net-(D2-Pad1) -> Net-(D18-Pad1)
- D18 pad 2: /Row1/High -> /Row4/High
- D19 pad 1: /Row1/Low -> /Row4/Low
- D19 pad 2: Net-(D2-Pad1) -> Net-(D18-Pad1)
- D20 pad 1: Net-(D2-Pad1) -> Net-(D20-Pad1)
- D20 pad 2: /Row1/High -> /Row5/High
- D21 pad 1: /Row1/Low -> /Row5/Low
- D21 pad 2: Net-(D2-Pad1) -> Net-(D20-Pad1)
- D22 pad 1: Net-(D2-Pad1) -> Net-(D22-Pad1)
- D23 pad 2: Net-(D2-Pad1) -> Net-(D22-Pad1)
- D24 pad 1: Net-(D2-Pad1) -> Net-(D24-Pad1)
- D24 pad 2: /Row1/High -> /Row2/High
- D25 pad 1: /Row1/Low -> /Row2/Low
- D25 pad 2: Net-(D2-Pad1) -> Net-(D24-Pad1)
- D26 pad 1: Net-(D2-Pad1) -> Net-(D26-Pad1)
- D26 pad 2: /Row1/High -> /Row3/High
- D27 pad 1: /Row1/Low -> /Row3/Low
- D27 pad 2: Net-(D2-Pad1) -> Net-(D26-Pad1)
- D28 pad 1: Net-(D2-Pad1) -> Net-(D28-Pad1)
- D28 pad 2: /Row1/High -> /Row4/High
- D29 pad 1: /Row1/Low -> /Row4/Low
- D29 pad 2: Net-(D2-Pad1) -> Net-(D28-Pad1)
- D30 pad 1: Net-(D2-Pad1) -> Net-(D30-Pad1)
- D30 pad 2: /Row1/High -> /Row5/High
- D31 pad 1: /Row1/Low -> /Row5/Low
- D31 pad 2: Net-(D2-Pad1) -> Net-(D30-Pad1)
- D32 pad 1: Net-(D2-Pad1) -> Net-(D32-Pad1)
- D33 pad 2: Net-(D2-Pad1) -> Net-(D32-Pad1)
- D34 pad 1: Net-(D2-Pad1) -> Net-(D34-Pad1)
- D34 pad 2: /Row1/High -> /Row2/High
- D35 pad 1: /Row1/Low -> /Row2/Low
- D35 pad 2: Net-(D2-Pad1) -> Net-(D34-Pad1)
- D36 pad 1: Net-(D2-Pad1) -> Net-(D36-Pad1)
- D36 pad 2: /Row1/High -> /Row3/High
- D37 pad 1: /Row1/Low -> /Row3/Low
- D37 pad 2: Net-(D2-Pad1) -> Net-(D36-Pad1)
- D38 pad 1: Net-(D2-Pad1) -> Net-(D38-Pad1)
- D38 pad 2: /Row1/High -> /Row4/High
- D39 pad 1: /Row1/Low -> /Row4/Low
- D39 pad 2: Net-(D2-Pad1) -> Net-(D38-Pad1)
- D4 pad 1: Net-(D2-Pad1) -> Net-(D4-Pad1)
- D4 pad 2: /Row1/High -> /Row2/High
- D40 pad 1: Net-(D2-Pad1) -> Net-(D40-Pad1)
- D40 pad 2: /Row1/High -> /Row5/High
- D41 pad 1: /Row1/Low -> /Row5/Low
- D41 pad 2: Net-(D2-Pad1) -> Net-(D40-Pad1)
- D42 pad 1: Net-(D2-Pad1) -> Net-(D42-Pad1)
- D43 pad 2: Net-(D2-Pad1) -> Net-(D42-Pad1)
- D44 pad 1: Net-(D2-Pad1) -> Net-(D44-Pad1)
- D44 pad 2: /Row1/High -> /Row2/High
- D45 pad 1: /Row1/Low -> /Row2/Low
- D45 pad 2: Net-(D2-Pad1) -> Net-(D44-Pad1)
- D46 pad 1: Net-(D2-Pad1) -> Net-(D46-Pad1)
- D46 pad 2: /Row1/High -> /Row3/High
- D47 pad 1: /Row1/Low -> /Row3/Low
- D47 pad 2: Net-(D2-Pad1) -> Net-(D46-Pad1)
- D48 pad 1: Net-(D2-Pad1) -> Net-(D48-Pad1)
- D48 pad 2: /Row1/High -> /Row4/High
- D49 pad 1: /Row1/Low -> /Row4/Low
- D49 pad 2: Net-(D2-Pad1) -> Net-(D48-Pad1)
- D5 pad 1: /Row1/Low -> /Row2/Low
- D5 pad 2: Net-(D2-Pad1) -> Net-(D4-Pad1)
- D50 pad 1: Net-(D2-Pad1) -> Net-(D50-Pad1)
- D50 pad 2: /Row1/High -> /Row5/High
- D51 pad 1: /Row1/Low -> /Row5/Low
- D51 pad 2: Net-(D2-Pad1) -> Net-(D50-Pad1)
- D52 pad 2: Net-(D52-Pad2) -> /GateDrive
- D55 pad 1: Net-(D55-Pad1) -> /Controller/IND_SR1_1
- D55 pad 2: +5V -> Net-(D55-Pad2)
- D56 pad 1: Net-(D56-Pad1) -> /Controller/IND_SR1_2
- D56 pad 2: +5V -> Net-(D56-Pad2)
- D57 pad 1: Net-(D57-Pad1) -> /Controller/IND_SR2
- D57 pad 2: +5V -> Net-(D57-Pad2)
- D58 pad 1: Net-(D58-Pad1) -> /Controller/IND_SR3
- D58 pad 2: +5V -> Net-(D58-Pad2)
- D6 pad 1: Net-(D2-Pad1) -> Net-(D6-Pad1)
- D6 pad 2: /Row1/High -> /Row3/High
- D7 pad 1: /Row1/Low -> /Row3/Low
- D7 pad 2: Net-(D2-Pad1) -> Net-(D6-Pad1)
- D8 pad 1: Net-(D2-Pad1) -> Net-(D8-Pad1)
- D8 pad 2: /Row1/High -> /Row4/High
- D9 pad 1: /Row1/Low -> /Row4/Low
- D9 pad 2: Net-(D2-Pad1) -> Net-(D8-Pad1)
- Px10 pad 1: Net-(D12-Pad1) -> Net-(D20-Pad1)
- Px12 pad 1: Net-(D22-Pad1) -> Net-(D24-Pad1)
- Px13 pad 1: Net-(D22-Pad1) -> Net-(D26-Pad1)
- Px14 pad 1: Net-(D22-Pad1) -> Net-(D28-Pad1)
- Px15 pad 1: Net-(D22-Pad1) -> Net-(D30-Pad1)
- Px17 pad 1: Net-(D32-Pad1) -> Net-(D34-Pad1)
- Px18 pad 1: Net-(D32-Pad1) -> Net-(D36-Pad1)
- Px19 pad 1: Net-(D32-Pad1) -> Net-(D38-Pad1)
- Px2 pad 1: Net-(D2-Pad1) -> Net-(D4-Pad1)
- Px20 pad 1: Net-(D32-Pad1) -> Net-(D40-Pad1)
- Px22 pad 1: Net-(D42-Pad1) -> Net-(D44-Pad1)
- Px23 pad 1: Net-(D42-Pad1) -> Net-(D46-Pad1)
- Px24 pad 1: Net-(D42-Pad1) -> Net-(D48-Pad1)
- Px25 pad 1: Net-(D42-Pad1) -> Net-(D50-Pad1)
- Px3 pad 1: Net-(D2-Pad1) -> Net-(D6-Pad1)
- Px4 pad 1: Net-(D2-Pad1) -> Net-(D8-Pad1)
- Px5 pad 1: Net-(D2-Pad1) -> Net-(D10-Pad1)
- Px7 pad 1: Net-(D12-Pad1) -> Net-(D14-Pad1)
- Px8 pad 1: Net-(D12-Pad1) -> Net-(D16-Pad1)
- Px9 pad 1: Net-(D12-Pad1) -> Net-(D18-Pad1)
- Q22 pad 2: MatrixControl1 -> MatrixControl2
- Q22 pad 4: MatrixControl2 -> MatrixControl1
- R15 pad 2: MatrixControl1 -> MatrixControl2
- R16 pad 2: MatrixControl2 -> MatrixControl1
- R26 pad 1: Net-(D55-Pad1) -> +3V3
- R26 pad 2: /Controller/IND_SR1_1 -> Net-(D55-Pad2)
- R27 pad 1: Net-(D56-Pad1) -> +3V3
- R27 pad 2: /Controller/IND_SR1_2 -> Net-(D56-Pad2)
- R28 pad 1: Net-(D57-Pad1) -> +3V3
- R28 pad 2: /Controller/IND_SR2 -> Net-(D57-Pad2)
- R29 pad 1: Net-(D58-Pad1) -> +3V3
- R29 pad 2: /Controller/IND_SR3 -> Net-(D58-Pad2)
- U6 pad 28: /Controller/storage_clock -> /Controller/data
- U6 pad 30: /Controller/data -> /Controller/storage_clock
- U7 pad 11: MatrixControl6 -> MatrixControl15
- U7 pad 12: MatrixControl5 -> MatrixControl16
- U7 pad 3: MatrixControl3 -> MatrixControl17
- U7 pad 4: MatrixControl4 -> MatrixControl18
- U7 pad 5: MatrixControl2 -> MatrixControl19
- U7 pad 6: MatrixControl1 -> MatrixControl20
- U8 pad 11: MatrixControl10 -> MatrixControl3
- U8 pad 12: MatrixControl11 -> MatrixControl1
- U8 pad 13: MatrixControl12 -> MatrixControl2
- U8 pad 3: MatrixControl13 -> MatrixControl11
- U8 pad 4: MatrixControl7 -> MatrixControl12
- U8 pad 5: MatrixControl8 -> MatrixControl13
- U8 pad 6: MatrixControl9 -> MatrixControl14
- U9 pad 11: MatrixControl16 -> MatrixControl10
- U9 pad 12: MatrixControl17 -> MatrixControl9
- U9 pad 13: MatrixControl18 -> MatrixControl8
- U9 pad 14: MatrixControl19 -> MatrixControl7
- U9 pad 4: MatrixControl20 -> MatrixControl6
- U9 pad 5: MatrixControl14 -> MatrixControl5
- U9 pad 6: MatrixControl15 -> MatrixControl4
Routing:
- net /Row1/Low: track 400.0 -> 80.0 mm
- net /Row1/High: track 400.0 -> 80.0 mm
- net MatrixControl9: track 2.06 -> 158.4 mm, vias 1 -> 2
- net MatrixControl10: track 2.06 -> 158.3 mm, vias 1 -> 2
- net MatrixControl7: track 2.06 -> 142.3 mm, vias 1 -> 2
- net MatrixControl8: track 2.06 -> 141.8 mm, vias 1 -> 2
- net Net-(D2-Pad1): track 105.0 -> 4.20 mm
- net MatrixControl4: track 10.3 -> 100.1 mm, vias 1 -> 2
- net MatrixControl5: track 29.9 -> 119.1 mm, vias 1 -> 2
- net MatrixControl6: track 33.4 -> 121.7 mm, vias 1 -> 2
- net MatrixControl3: track 7.41 -> 95.0 mm, vias 1 -> 2
- net MatrixControl20: track 2.06 -> 88.3 mm, vias 1 -> 3
- net MatrixControl19: track 2.06 -> 86.2 mm, vias 1 -> 3
- net +3V3: track 5.01 -> 86.4 mm, vias 0 -> 9
- net /Row5/Low: track 0.00 -> 80.0 mm
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- added copper zone on F.Cu, net +5V
- added copper zone on B.Cu, net /PixelMatrix/Col_1
- added copper zone on B.Cu, net /PixelMatrix/Col_2
- added copper zone on B.Cu, net /PixelMatrix/Col_3
- added copper zone on B.Cu, net /PixelMatrix/Col_4
- added copper zone on B.Cu, net /PixelMatrix/Col_5
- added copper zone on F.Cu, net /Row2/High
- added copper zone on F.Cu, net /Row2/Low
- added copper zone on F.Cu, net /Row3/High
- added copper zone on F.Cu, net /Row3/Low
- added copper zone on F.Cu, net /Row4/High
- added copper zone on F.Cu, net /Row4/Low
- added copper zone on F.Cu, net /Row5/High
- added copper zone on F.Cu, net /Row5/Low
- added copper zone on B.Cu, net MatrixPower
Other:
- board text added: "Flip Pixel Display Evaluation Board v0.2"
- board text removed: "Flip Pixel Display Evaluation Board Spin 1"

Commit message: Ready for Manufacture
Parts:
- added H1: MountingHole, MountingHole:MountingHole_3mm, F.Cu at (112.0, 51.0)
- added H2: MountingHole, MountingHole:MountingHole_3mm, F.Cu at (219.0, 51.0)
- added H3: MountingHole, MountingHole:MountingHole_3mm, F.Cu at (219.0, 150.0)
- added H4: MountingHole, MountingHole:MountingHole_3mm, F.Cu at (120.0, 150.0)
- added TP5: TestPoint, TestPoint:TestPoint_Pad_D2.0mm, B.Cu at (89.1, 117.2)
- added TP6: TestPoint, TestPoint:TestPoint_Pad_D2.0mm, B.Cu at (93.1, 117.2)
- moved TP1 86.5 mm to (93.0, 113.0)
- moved TP2 86.5 mm to (93.0, 109.0)
- moved TP3 86.5 mm to (89.0, 113.0)
- moved TP4 86.5 mm to (89.0, 109.0)
- moved J2 34.0 mm to (71.5, 132.3)
- moved C7 33.8 mm to (91.2, 135.2)
- moved C8 33.8 mm to (91.2, 133.1)
- moved U2 33.8 mm to (91.2, 138.3)
- moved C1 33.8 mm to (109.0, 145.8)
- moved C10 33.8 mm to (96.5, 105.7)
- moved C11 33.8 mm to (81.8, 134.2)
- moved C12 33.8 mm to (77.3, 121.8)
- moved C2 33.8 mm to (109.0, 142.3)
- moved C3 33.8 mm to (103.8, 119.0)
- moved C4 33.8 mm to (107.0, 115.4)
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Connections:
- C2 pad 1: /Power/matrix_current -> /Controller/matrix_current
- U4 pad 9: /Power/matrix_current -> /Controller/matrix_current
- U6 pad 36: /Controller/scl -> /Controller/SCL
- U6 pad 37: /Controller/sda -> /Controller/SDA
Routing:
- net /Controller/matrix_current: track 0.00 -> 33.6 mm, vias 0 -> 3
- net +3V3: track 86.4 -> 117.2 mm
- net +5V: track 13.3 -> 35.1 mm, vias 1 -> 3
- net /Controller/esp_tx: track 33.8 -> 51.9 mm, vias 0 -> 1
- net /Controller/SDA: track 0.00 -> 16.0 mm, vias 0 -> 1
- net /Controller/esp_rx: track 33.3 -> 46.9 mm, vias 0 -> 1
- net /Controller/SCL: track 0.00 -> 12.7 mm, vias 0 -> 1
- net /Power/matrix_current: track 3.38 -> 0.00 mm, vias 1 -> 0
- net MatrixControl2: track 80.3 -> 77.2 mm
- net GND: track 60.9 -> 63.8 mm
- net MatrixControl1: track 78.2 -> 76.7 mm
Other:
- board size 151.4 x 100.4 mm -> 154 x 107 mm

Commit message: small tweaks and version migration
Parts:
- added J3: Conn_01x07_Female, Connector_PinSocket_2.54mm:PinSocket_1x07_P2.54mm_Vertical, F.Cu at (73.0, 62.9)
- added R31: R, Resistor_SMD:R_0805_2012Metric, F.Cu at (109.6, 128.1)
- added R32: R, Resistor_SMD:R_0805_2012Metric, F.Cu at (109.6, 130.2)
- added TP7: TestPoint, TestPoint:TestPoint_Pad_D2.0mm, F.Cu at (108.7, 124.3)
- moved J2 0.24 mm to (71.7, 132.2)
Connections:
- net /Controller/matrix_current renamed /matrix_current
- net /Controller/usb_D+ renamed /usb_D+
- net /Controller/usb_D- renamed /usb_D-
- net /PixelMatrix/Col_1 renamed /Low_1
- net /PixelMatrix/Col_2 renamed /High_4
- net /PixelMatrix/Col_3 renamed /Col_3
- net /PixelMatrix/Col_4 renamed /High_3
- net /PixelMatrix/Col_5 renamed /High_2
- net /Power/10V_enable renamed /matrix_enable
- net /Row1/High renamed /High
- net /Row1/Low renamed /Row_1_L
- net /Row2/High renamed /Row_2_H
- net /Row2/Low renamed /Low
- net /Row3/High renamed /High_1
- net /Row3/Low renamed /Row_3_L
- net /Row4/High renamed /Row_4_H
- net /Row4/Low renamed /Row_4_L
- net /Row5/High renamed /Row_5_H
- net /Row5/Low renamed /Row_5_L
- U5 pad 11: Net-(U5-Pad11) -> +3V3
Routing:
- net /matrix_enable: track 30.3 -> 95.5 mm, vias 2 -> 4
- net /Controller/data: track 10.7 -> 51.6 mm, vias 0 -> 2
- net /Controller/~output_enable: track 31.3 -> 59.6 mm, vias 3 -> 4
- net /Controller/~master_reset: track 31.4 -> 56.7 mm, vias 3 -> 4
- net +3V3: track 117.2 -> 126.0 mm, vias 9 -> 10
- net /Controller/shift_clock: track 51.8 -> 58.5 mm
- net Net-(R31-Pad2): track 0.00 -> 5.95 mm
- net /Controller/storage_clock: track 78.3 -> 83.3 mm
- net GND: track 63.8 -> 61.0 mm, vias 32 -> 33
- net MatrixPower: track 1.30 -> 3.03 mm
- net MatrixControl13: track 51.5 -> 50.6 mm
Other:
- net class Default removed
